File: ECAD/MainBoard-PAMI-2024/MainBoard-PAMI-2024.kicad_pcb (KiCad board)
At the start: 2 copper layers, 79.5 x 96 mm, 48 parts, among them J1 Selecteur-Robot, J10 Serial, J11 Con_Batt, J12 BAU, J2 USB_B, J3 Tirette, J4 Servo, J5 Sensor_Right, J6 Sensor_Left, J7 LeftMotor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

Commit message: First routing
Parts:
- removed BZ1: Buzzer, Buzzer_Beeper:Buzzer_12x9.5RM7.6
- removed J9: color_team, Connector_Molex:Molex_KK-254_AE-6410-02A_1x02_P2.54mm_Vertical
- added J13: OLED, Connector_Molex:Molex_KK-254_AE-6410-04A_1x04_P2.54mm_Vertical, F.Cu at (128.5, 66.8)
- added R10: 10K, Resistor_SMD:R_1206_3216Metric_Pad1.30x1.75mm_HandSolder, F.Cu at (132.6, 71.5)
- added R11: 10K, Resistor_SMD:R_1206_3216Metric_Pad1.30x1.75mm_HandSolder, F.Cu at (130.0, 74.2)
- added SW1: SW_SPDT, footprints:SK-12D10 1P2T, F.Cu at (127.0, 58.0)
- J11: footprint Connector_Molex:Molex_KK-254_AE-6410-02A_1x02_P2.54mm_Vertical -> Connector_AMASS:AMASS_XT30U-F_1x02_P5.0mm_Vertical
- J12: footprint Connector_Molex:Molex_KK-254_AE-6410-02A_1x02_P2.54mm_Vertical -> Connector_Molex:Molex_KK-396_A-41791-0002_1x02_P3.96mm_Vertical
- R7, R8: value 4K7 -> 10K
- moved R7 70.0 mm to (104.8, 137.2)
- moved R8 70.0 mm to (104.8, 134.6)
- moved C5 38.0 mm to (125.3, 110.2), turned to 90 degrees
- moved SWBoot1 29.6 mm to (128.8, 112.6)
- moved R6 23.0 mm to (117.9, 105.9), turned to 180 degrees
- moved D3 19.7 mm to (155.2, 120.6)
- moved R1 14.8 mm to (155.2, 123.2)
- moved D6 10.6 mm to (153.5, 126.5), turned to -90 degrees
- moved C10 10.3 mm to (159.8, 79.0)
- moved J3 9.80 mm to (141.9, 109.2), turned to 180 degrees
- moved C1 7.40 mm to (148.2, 75.2)
- moved D4 7.37 mm to (170.4, 73.7)
- moved D5 7.37 mm to (170.4, 71.1)
- moved D8 7.37 mm to (170.4, 76.2)
- moved R2 7.37 mm to (164.7, 73.7)
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Connections:
- net Net-(D6-A) renamed /D+
- net Net-(D7-A) renamed /D-
- J11 pad 1: GND -> +BATT
- J11 pad 2: +BATT -> GND
- U1 pad 36: Net-(J10-Pin_1) -> Net-(J10-Pin_2)
- U1 pad 37: Net-(J10-Pin_2) -> Net-(J10-Pin_1)
Routing:
- net +3.3V: track 0.00 -> 239.3 mm, vias 0 -> 1
- net +5VP: track 0.00 -> 151.4 mm
- net SCL: track 0.00 -> 149.6 mm, vias 0 -> 1
- net SDA: track 0.00 -> 141.5 mm, vias 0 -> 2
- net Color_Team: track 0.00 -> 87.8 mm, vias 0 -> 3
- net XSHUT_RIGHT: track 0.00 -> 80.1 mm, vias 0 -> 3
- net LED_Status: track 0.00 -> 63.4 mm, vias 0 -> 2
- net RightDir: track 0.00 -> 61.0 mm
- net LeftMS2: track 0.00 -> 59.6 mm, vias 0 -> 1
- net RightStep: track 0.00 -> 58.0 mm
- net LeftMS1: track 0.00 -> 56.7 mm, vias 0 -> 1
- net EnDriver: track 0.00 -> 53.5 mm, vias 0 -> 1
- net +BATT: track 0.00 -> 37.6 mm, vias 0 -> 1
- net Servo: track 0.00 -> 29.4 mm, vias 0 -> 2
- net XSHUT_LEFT: track 0.00 -> 28.8 mm
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
Commit message: Fix XT60 (Histo t'as vu)
Parts:
- moved J11 4.60 mm to (141.5, 92.6), turned to 180 degrees
Connections:
- J11 pad 1: +BATT -> GND
- J11 pad 2: GND -> +BATT
Changed lines of the file:
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@@
   )
   (footprint "Connector_AMASS:AMASS_XT30U-F_1x02_P5.0mm_Vertical" (layer "F.Cu")
-    (at 136.9 92.6)
+    (at 141.5 92.6 180)
     (descr "Connector XT30 Vertical Cable Female, https://www.tme.eu/en/Document/3cbfa5cfa544d79584972dd5234a409e/XT30U%20SPEC.pdf")
     (tags "RC Connector XT30")
@@
     (property "ki_keywords" "connector")
     (attr through_hole)
-    (fp_text reference "J11" (at 2.9 -2 180) (layer "F.SilkS")
+    (fp_text reference "J11" (at 2.9 -2) (layer "F.SilkS")
         (effects (font (size 0.6 0.6) (thickness 0.15)))
     )
@@
     (fp_line (start 7.6 -2.6) (end 7.6 2.6)
       (stroke (width 0.1) (type solid)) (layer "F.Fab"))
-    (pad "1" thru_hole rect (at 0 0) (size 3.8 3.8) (drill 2.7) (layers "*.Cu" "*.Mask")
-      (net 67 "+BATT") (pinfunction "Pin_1") (pintype "passive"))
-    (pad "2" thru_hole circle (at 5 0) (size 4 4) (drill 2.7) (layers "*.Cu" "*.Mask")
-      (net 1 "GND") (pinfunction "Pin_2") (pintype "passive"))
+    (pad "1" thru_hole rect (at 0 0 180) (size 3.8 3.8) (drill 2.7) (layers "*.Cu" "*.Mask")
+      (net 1 "GND") (pinfunction "Pin_1") (pintype "passive"))
+    (pad "2" thru_hole circle (at 5 0 180) (size 4 4) (drill 2.7) (layers "*.Cu" "*.Mask")
+      (net 67 "+BATT") (pinfunction "Pin_2") (pintype "passive"))
     (model "${KIPRJMOD}/Packages3D/AMASS_XT30U-F_1x02_P5.0mm_Vertical.wrl"
       (offset (xyz 0 0 0))
@@
   (segment (start 163.169 78.333) (end 163.576 78.74) (width 1) (layer "F.Cu") (net 67))
   (via (at 163.576 78.74) (size 0.8) (drill 0.4) (layers "F.Cu" "B.Cu") (net 67))
-  (segment (start 136.9 92.6) (end 136.9 88.46) (width 2.4) (layer "B.Cu") (net 67))
+  (segment (start 136.5 88.86) (end 139.6 85.76) (width 2.4) (layer "B.Cu") (net 67))
   (segment (start 163.576 78.74) (end 149.098 78.74) (width 1) (layer "B.Cu") (net 67))
   (segment (start 142.078 85.76) (end 139.6 85.76) (width 1) (layer "B.Cu") (net 67))
   (segment (start 149.098 78.74) (end 142.078 85.76) (width 1) (layer "B.Cu") (net 67))
-  (segment (start 136.9 88.46) (end 139.6 85.76) (width 2.4) (layer "B.Cu") (net 67))
+  (segment (start 136.5 92.2) (end 136.5 88.86) (width 2.4) (layer "B.Cu") (net 67))
   (segment (start 166.269 76.2) (end 169.034 76.2) (width 1) (layer "F.Cu") (net 68))
   (segment (start 153.017999 127.192) (end 153.543 127.192) (width 0.25) (layer "F.Cu") (net 69))

Commit message: Silkscreen
Parts:
- added G***: LOGO, LOGO, F.Cu at (121.7, 141.8)
- added G***: LOGO, LOGO, F.Cu at (104.5, 99.9)
- added G***: LOGO, LOGO, F.Cu at (107.2, 129.3)
- added G***: LOGO, LOGO, F.Cu at (105.2, 93.9)
- added G***: LOGO, LOGO, F.Cu at (106.9, 114.1)
- added G***: LOGO, LOGO, B.Cu at (138.2, 66.8)
- added G***: LOGO, LOGO, B.Cu at (110.0, 136.0)
- added G***: LOGO, LOGO, B.Cu at (106.6, 58.0)
- added G***: LOGO, LOGO, B.Cu at (121.7, 141.8)
- added G***: LOGO, LOGO, B.Cu at (136.9, 109.2)
- added G***: LOGO, LOGO, B.Cu at (106.9, 71.1)
- added G***: LOGO, LOGO, F.Cu at (110.0, 136.0)
- added G***: LOGO, LOGO, B.Cu at (106.8, 142.2)
- added G***: LOGO, LOGO, B.Cu at (163.6, 125.8)
- added G***: LOGO, LOGO, B.Cu at (107.2, 129.3)
- added G***: LOGO, LOGO, B.Cu at (109.0, 109.2)
- added G***: LOGO, LOGO, B.Cu at (106.9, 86.4)
- added G***: LOGO, LOGO, B.Cu at (106.9, 114.1)
- added G***: LOGO, LOGO, F.Cu at (106.9, 86.4)
- added G***: LOGO, LOGO, F.Cu at (138.2, 66.8)
- added G***: LOGO, LOGO, F.Cu at (136.9, 109.2)
- added G***: LOGO, LOGO, F.Cu at (106.9, 71.1)
- added G***: LOGO, LOGO, F.Cu at (109.0, 109.2)
- added G***: LOGO, LOGO, F.Cu at (129.1, 93.5)
- added G***: LOGO, LOGO, F.Cu at (106.6, 58.0)
- added H3: MountingHole, MountingHole:MountingHole_3.2mm_M3, F.Cu at (162.9, 139.0)
- added kibuzzard-65231966: G***, kibuzzard-65231966, F.Cu at (105.5, 131.9)
- added kibuzzard-65231966: G***, kibuzzard-65231966, F.Cu at (113.8, 105.5)
- added kibuzzard-65231966: G***, kibuzzard-65231966, F.Cu at (105.5, 88.9)
- added kibuzzard-65231966: G***, kibuzzard-65231966, B.Cu at (105.5, 88.9)
- added kibuzzard-65231966: G***, kibuzzard-65231966, B.Cu at (139.6, 77.5)
- added kibuzzard-65231966: G***, kibuzzard-65231966, B.Cu at (105.5, 131.9)
- added kibuzzard-654226B4: G***, kibuzzard-654226B4, F.Cu at (133.7, 63.8)
- added kibuzzard-654226B4: G***, kibuzzard-654226B4, F.Cu at (106.2, 116.6)
- added kibuzzard-654226B4: G***, kibuzzard-654226B4, F.Cu at (106.2, 73.6)
- added kibuzzard-654226B4: G***, kibuzzard-654226B4, F.Cu at (106.0, 60.5)
- added kibuzzard-654226B4: G***, kibuzzard-654226B4, B.Cu at (105.8, 144.9)
- added kibuzzard-654226B4: G***, kibuzzard-654226B4, B.Cu at (106.0, 60.5)
- added kibuzzard-654226B4: G***, kibuzzard-654226B4, B.Cu at (106.2, 116.6)
- added kibuzzard-654226B4: G***, kibuzzard-654226B4, B.Cu at (106.2, 73.6)
- added kibuzzard-654226B4: G***, kibuzzard-654226B4, B.Cu at (133.7, 63.8)
- added kibuzzard-65422827: G***, kibuzzard-65422827, F.Cu at (114.2, 64.8)
- added kibuzzard-6542284D: G***, kibuzzard-6542284D, F.Cu at (122.7, 62.2)
- added kibuzzard-65422864: G***, kibuzzard-65422864, F.Cu at (126.2, 66.6)
- added kibuzzard-65422975: G***, kibuzzard-65422975, F.Cu at (133.7, 83.6)
- added kibuzzard-65422987: G***, kibuzzard-65422987, F.Cu at (136.6, 96.1)
- added kibuzzard-6542299D: G***, kibuzzard-6542299D, F.Cu at (140.3, 113.0)
- added kibuzzard-654229BB: G***, kibuzzard-654229BB, F.Cu at (119.8, 109.2)
- added kibuzzard-65422A0E: G***, kibuzzard-65422A0E, F.Cu at (131.8, 112.7)
- added kibuzzard-65422A22: G***, kibuzzard-65422A22, F.Cu at (149.8, 118.0)
- added kibuzzard-65422AAE: G***, kibuzzard-65422AAE, F.Cu at (159.3, 71.1)
- added kibuzzard-65422AB6: G***, kibuzzard-65422AB6, F.Cu at (160.2, 73.7)
- added kibuzzard-65422AC7: G***, kibuzzard-65422AC7, F.Cu at (159.8, 76.2)
- added kibuzzard-65422F57: G***, kibuzzard-65422F57, F.Cu at (126.2, 93.8)
- added kibuzzard-65423033: G***, kibuzzard-65423033, F.Cu at (123.2, 134.8)
- added kibuzzard-65423064: G***, kibuzzard-65423064, F.Cu at (126.3, 136.9)
- added kibuzzard-65423077: G***, kibuzzard-65423077, F.Cu at (126.3, 139.4)
- added kibuzzard-654230EB: G***, kibuzzard-654230EB, F.Cu at (114.3, 138.2)
- added kibuzzard-6542315C: G***, kibuzzard-6542315C, F.Cu at (116.8, 138.2)
- added kibuzzard-65423198: G***, kibuzzard-65423198, F.Cu at (124.6, 129.3)
- added kibuzzard-65423198: G***, kibuzzard-65423198, F.Cu at (124.7, 86.3)
- added kibuzzard-654231C8: G***, kibuzzard-654231C8, F.Cu at (124.6, 114.1)
- added kibuzzard-654231C8: G***, kibuzzard-654231C8, F.Cu at (124.7, 71.1)
- added kibuzzard-654231D0: G***, kibuzzard-654231D0, F.Cu at (124.7, 73.7)
- added kibuzzard-654231D0: G***, kibuzzard-654231D0, F.Cu at (124.6, 116.7)
- added kibuzzard-654231D6: G***, kibuzzard-654231D6, F.Cu at (124.7, 83.8)
- added kibuzzard-654231D6: G***, kibuzzard-654231D6, F.Cu at (124.6, 126.8)
- added kibuzzard-654231DD: G***, kibuzzard-654231DD, F.Cu at (124.7, 88.9)
- added kibuzzard-654231DD: G***, kibuzzard-654231DD, F.Cu at (124.6, 131.9)
Connections:
- net Net-(J10-Pin_1) renamed /TX
- net Net-(J10-Pin_2) renamed /RX
Other:
- board text added: "Karibous 2023-24 Barbatronic"
- board text added: "PAMI - 2024 Main Board"
